File: KiCAD/DoughLee2.kicad_pcb (KiCad board)
At the start: 4 copper layers, 69.8 x 44.5 mm, 63 parts, among them J1 Conn_01x06, J3 Edge2x6_Connector, U1 SHTC3, U2 ESP32-WROOM-32, U3 AMS1117-3.3, U4 SN74LVC1G123DCUR, U5 74LVC1G08

Commit message: Updated KiCAD design
- Fix library locations
- Update some footprints and symbols
- Added missing +3.3V to SHTC3
- Removed jumper from edge-connector power and replaced with wire
Parts:
- removed the JP1 at (94.6, 61.6)
- DHR1: footprint Diode_SMD:D_SMA -> Diode_SMD:D_SMB
- J3: footprint Library:EdgeConnector_2x3 -> chl33_library:EdgeConnector_2x3
- L1: value 100 μH -> 100 μH; footprint Library:CD54 -> chl33_library:CD54
- U4: footprint Library:SOP50P310X90-8N -> chl33_library:SOP50P310X90-8N
- U5: footprint Library:SOT-23-5 -> chl33_library:SOT-23-5
- U_B1: footprint Library:BD90610EFJ-CE2 -> chl33_library:BD90610EFJ-CE2
Connections:
- C2 pad 1: +5V -> VBUS
- Cb3 pad 1: +5V -> VBUS
- Cc2 pad 1: +5V -> VBUS
- J1 pad 3: +5V -> VBUS
- L1 pad 2: +5V -> VBUS
- RB2 pad 1: +5V -> VBUS
- U3 pad 3: +5V -> VBUS
Routing:
- net VBUS: track 7.07 -> 85.9 mm, vias 1 -> 5
- net +5V: track 77.5 -> 0.00 mm, vias 4 -> 0
- net +3.3V: track 113.1 -> 114.7 mm
Other:
- outline, holes or cut-outs redrawn
- board text added: "DoughLee v3.6 (c) Chris Lee"
- board text removed: "DoughLee v3.5 (c) Chris Lee"
