File: KiCAD/ESP32-NoSerial.kicad_sch (KiCad schematic)
At the start: 10 parts, among them J3 Edge2x6_Connector, U2 ESP32-WROOM-32, U3 AMS1117-3.3

Commit message: Updated KiCAD design
- Fix library locations
- Update some footprints and symbols
- Added missing +3.3V to SHTC3
- Removed jumper from edge-connector power and replaced with wire
Parts:
- J3: footprint Library:EdgeConnector_2x3 -> chl33_library:EdgeConnector_2x3
