File: KiCAD/buck5v.kicad_sch (KiCad schematic)
At the start: 13 parts

Commit message: Updated KiCAD design
- Fix library locations
- Update some footprints and symbols
- Added missing +3.3V to SHTC3
- Removed jumper from edge-connector power and replaced with wire
Parts:
- L1: value 100 μH -> 100 μH; footprint Library:CD54 -> chl33_library:CD54
